Commit message: rearranging launch files and frame ids to match closer to pensa's stack

File: urdf/cinderella_new.urdf (robot description, URDF)
Before this commit: robot cinderella_3d, 4 links, 3 joints
Links:
- removed link odom_frame
- added link base_link_vislam
Joints:
- joint odom_link_joint: parent odom_frame -> base_link_vislam

Commit message: updates on lidar topic and frame_id

File: urdf/cinderella_new.urdf (robot description, URDF)
Before this commit: robot cinderella_3d, 4 links, 3 joints
Links:
- removed link laser_frame
- added link laser_hector_frame; visual cylinder length=0.07 radius=0.05
Joints:
- joint lidar_link_joint: child laser_frame -> laser_hector_frame
